Commit message: adding diff_driver controller

File: vc200_description/urdf/macros/wheel.xacro (robot description, xacro)
@@ -3,4 +3,10 @@
     <xacro:macro name="wheel" params="name radius width dx dy">
         <link name="${name}_link">
+            <collision>
+                <origin xyz="0 0 0" rpy="0 0 0" />
+                <geometry>
+                    <cylinder radius="${radius}" length="${width}" />
+                </geometry>
+            </collision>
             <visual>
                 <origin xyz="0.0 0.0 0.0" rpy="0.0 0.0 0.0" />
