Commit message: adding localization update

File: vc200_description/urdf/macros/imu.xacro (robot description, xacro)
@@ -1,5 +1,5 @@
 <?xml version="1.0"?>
 <robot xmlns:xacro="http://www.ros.org/wiki/xacro">
-    <xacro:macro name="pozyx" params="name length width height dx dy dz ar ap ay">
+    <xacro:macro name="imu" params="name length width height dx dy dz ar ap ay">
         <link name="${name}_link">
             <collision>
@@ -14,5 +14,5 @@
                     <box size="${length} ${width} ${height}" />
                 </geometry>
-                <material name="pozyx" />
+                <material name="imu" />
             </visual>
         </link>

File: vc200_description/urdf/macros/macros.xacro (robot description, xacro)
@@ -7,3 +7,4 @@
     <xacro:include filename="$(find vc200_description)/urdf/macros/marvelmind.xacro" />
     <xacro:include filename="$(find vc200_description)/urdf/macros/lidar.xacro" />
+    <xacro:include filename="$(find vc200_description)/urdf/macros/imu.xacro" />
 </robot>

File: vc200_description/urdf/macros/materials.xacro (robot description, xacro)
@@ -16,3 +16,6 @@
         <color rgba="1 1 1 1.0"/>
     </material>
+    <material name="imu">
+        <color rgba="1 1 1 1.0"/>
+    </material>
 </robot>

File: vc200_description/urdf/parameters.xacro (robot description, xacro)
@@ -13,4 +13,3 @@
     <xacro:property name="wheel_separation" value="0.3"/>
     <xacro:property name="wheelbase" value="0.24"/>
-    wheelbase
 </robot>

File: vc200_description/urdf/vc200_description.xacro (robot description, xacro)
@@ -1,5 +1,5 @@
 <?xml version="1.0"?>
-<!-- <robot name="$(arg robot_name)" xmlns:xacro="http://www.ros.org/wiki/xacro"> -->
-<robot name="vc200" xmlns:xacro="http://www.ros.org/wiki/xacro">
+<robot name="$(arg robot_name)" xmlns:xacro="http://www.ros.org/wiki/xacro">
+<!-- <robot name="vc200" xmlns:xacro="http://www.ros.org/wiki/xacro"> -->
     <xacro:include filename="$(find vc200_description)/urdf/parameters.xacro" />
     <xacro:include filename="$(find vc200_description)/urdf/macros/macros.xacro" />
@@ -49,5 +49,5 @@
       ar="0.0"
       ap="0.0"
-      ay="0.0"
+      ay="${PI}"
     />
     <!-- radius="0.035"
@@ -60,7 +60,10 @@
       dx="-0.025"
       dy="0.045"
-      dz="${0.12+clearence+0.003/3}"
+      dz="${0.12+clearence+0.003/2}"
+      ar="0.0"
+      ap="0.0"
+      ay="0.0"
     />
-    <xacro:marvelmind
+    <!-- <xacro:marvelmind
       name="${robot_name}/marvelmind"
       length ="0.055"
@@ -73,4 +76,16 @@
       ap="0.69813170079"
       ay="0.0"
+    /> -->
+    <xacro:imu
+      name="${robot_name}/stm_imu"
+      length="0.008"
+      width="0.006"
+      height="0.003"
+      dx="-0.025"
+      dy="0.045"
+      dz="${0.12+clearence+0.003/2 - 0.02}"
+      ar="0.0"
+      ap="0.0"
+      ay="${-PI/2}"
     />
     <xacro:arg name="use_nominal_extrinsics" default="true" />
