Commit message: Added lidar and world config with house

File: vc200_description/urdf/macros/lidar.xacro (robot description, xacro)
@@ -1,18 +1,27 @@
 <?xml version="1.0"?>
 <robot xmlns:xacro="http://www.ros.org/wiki/xacro">
-    <xacro:macro name="lidar" params="name radius length dx dy dz ar ap ay">
+    <xacro:macro name="lidar" params="name radius height *origin mass">
         <link name="${name}_link">
             <visual>
                 <origin xyz="0.0 0.0 0.0" rpy="0.0 0.0 0.0" />
                 <geometry>
-                    <cylinder radius="${radius}" length="${length}" />
+                    <cylinder radius="${radius}" length="${height}" />
                 </geometry>
                 <material name="lidar" />
             </visual>
+            <collision name="${name}">
+                <origin xyz="0.0 0.0 0.0" rpy="0.0 0.0 0.0" />
+                <geometry>
+                    <cylinder radius="${radius}" length="${height}" />
+                </geometry>
+            </collision>
+            <xacro:cylinder_inertia radius="${radius}" length="${height}" mass="${mass}">
+                <origin xyz="0.0 0.0 0.0" rpy="0.0 0.0 0.0" />
+            </xacro:cylinder_inertia>
         </link>
         <joint name="${name}_joint" type="fixed">
             <parent link="${robot_name}/base_footprint" />
             <child link="${name}_link" />
-            <origin xyz="${dx} ${dy} ${dz}" rpy="${ar} ${ap} ${ay}" />
+            <xacro:insert_block name="origin" />
         </joint>
     </xacro:macro>

File: vc200_description/urdf/macros/macros.xacro (robot description, xacro)
@@ -10,3 +10,5 @@
     <xacro:include filename="$(find vc200_description)/urdf/macros/caster_wheel.xacro" />
     <xacro:include filename="$(find vc200_description)/urdf/macros/inertia.xacro" />
+    <!-- gazebo -->
+    <xacro:include filename="$(find vc200_description)/urdf/gazebo/lidar_sensor.xacro" />
 </robot>

File: vc200_description/urdf/vc200.gazebo.xacro (robot description, xacro)
@@ -39,4 +39,10 @@
     dx="${wheelbase/2.0}"
     dy="-${wheel_separation/2.0}" />
+  <xacro:lidar name="${robot_name}/rplidar"
+    radius="0.035"
+    height="0.03"
+    mass="0.17" >
+    <origin xyz="0.1 0.0 ${0.015+chassis_height+clearence}" rpy="0.0 0.0 0.0"/>
+  </xacro:lidar>
   <xacro:macro name="wheel_friction" params="friction">
     <mu1 value="${friction}" />
@@ -82,4 +88,12 @@
     </plugin>
   </gazebo>
+  <xacro:lidar_sensor
+  reference="${robot_name}/rplidar_link"
+  name="rplidar"
+  frame_id="${robot_name}/rplidar_link"
+  update_rate="40"
+  samples="720"
+  visualize="true"
+  type_prefix="gpu_" />
   <!-- <gazebo>
     <plugin name="gazebo_ros_control" filename="libgazebo_ros_control.so">
