Commit message: setup for two wheel platform

File: vc200_description/urdf/macros/macros.xacro (robot description, xacro)
@@ -8,3 +8,5 @@
     <xacro:include filename="$(find vc200_description)/urdf/macros/lidar.xacro" />
     <xacro:include filename="$(find vc200_description)/urdf/macros/imu.xacro" />
+    <xacro:include filename="$(find vc200_description)/urdf/macros/caster_wheel.xacro" />
+    <xacro:include filename="$(find vc200_description)/urdf/macros/inertia.xacro" />
 </robot>

File: vc200_description/urdf/parameters.xacro (robot description, xacro)
@@ -8,8 +8,13 @@
     <xacro:property name="chassis_width" value="0.18" />
     <xacro:property name="chassis_height" value="0.108" />
+    <xacro:property name="chassis_mass" value="0.5" /> <!-- TODO -->
     <xacro:property name="clearence" value="0.042" />
     <xacro:property name="wheel_radius" value="0.0675" />
+    <xacro:property name="wheel_mass" value="0.1" /> <!-- TODO -->
     <xacro:property name="wheel_width" value="0.057" />
-    <xacro:property name="wheel_separation" value="0.3"/>
-    <xacro:property name="wheelbase" value="0.24"/>
+    <xacro:property name="wheel_separation" value="0.3" />
+    <xacro:property name="wheelbase" value="0.24" />
+    <xacro:property name="update_rate" value="50" />
+    <!-- <xacro:property name="odometry_source" value="encoder" /> -->
+    <!-- <xacro:property name="odometry_source" value="world" /> -->
 </robot>

File: vc200_description/urdf/vc200_description.xacro (robot description, xacro)
@@ -1,5 +1,5 @@
 <?xml version="1.0"?>
-<robot name="$(arg robot_name)" xmlns:xacro="http://www.ros.org/wiki/xacro">
-<!-- <robot name="vc200" xmlns:xacro="http://www.ros.org/wiki/xacro"> -->
+<!-- <robot name="$(arg robot_name)" xmlns:xacro="http://www.ros.org/wiki/xacro"> -->
+<robot name="vc200" xmlns:xacro="http://www.ros.org/wiki/xacro">
     <xacro:include filename="$(find vc200_description)/urdf/parameters.xacro" />
     <xacro:include filename="$(find vc200_description)/urdf/macros/macros.xacro" />
@@ -11,33 +11,38 @@
       height="${chassis_height}"
       clearence="${clearence}"
+      mass="${chassis_mass}"
     />
     <xacro:wheel
-      name="${robot_name}/front_left_wheel"
+      name="${robot_name}/left_wheel"
       radius="${wheel_radius}"
       width="${wheel_width}"
+      mass="${wheel_mass}"
       dx="${wheelbase/2.0}"
       dy="${wheel_separation/2.0}"
     />
     <xacro:wheel
-      name="${robot_name}/front_right_wheel"
+      name="${robot_name}/right_wheel"
       radius="${wheel_radius}"
+      mass="${wheel_mass}"
       width="${wheel_width}"
       dx="${wheelbase/2.0}"
       dy="-${wheel_separation/2.0}"
     />
-    <xacro:wheel
-      name="${robot_name}/rear_left_wheel"
-      radius="${wheel_radius}"
-      width="${wheel_width}"
-      dx="-${wheelbase/2.0}"
-      dy="${wheel_separation/2.0}"
-    />
-    <xacro:wheel
-      name="${robot_name}/rear_right_wheel"
-      radius="${wheel_radius}"
-      width="${wheel_width}"
-      dx="-${wheelbase/2.0}"
-      dy="-${wheel_separation/2.0}"
-    />
+    <xacro:caster_wheel name="${robot_name}/caster_right"
+    radius="0.0125"
+    mass="0.01"
+    dx="-0.15"
+    dy="-0.05"
+    offset="0.014"
+    height="0.035"
+    width="0.007" />
+  <xacro:caster_wheel name="${robot_name}/caster_left"
+    radius="0.0125"
+    mass="0.01"
+    dx="-0.15"
+    dy="0.05"
+    offset="0.014"
+    height="0.035"
+    width="0.007" />
     <xacro:lidar
       name="${robot_name}/lidar"
@@ -65,5 +70,5 @@
       ay="0.0"
     />
-    <xacro:marvelmind
+    <!-- <xacro:marvelmind
       name="${robot_name}/marvelmind"
       length ="0.055"
@@ -76,5 +81,5 @@
       ap="0.69813170079"
       ay="0.0"
-    />
+    /> -->
     <xacro:imu
       name="${robot_name}/stm_imu"
