Commit message: parameters update

File: vc200_description/urdf/macros/caster_wheel.xacro (robot description, xacro)
@@ -46,5 +46,5 @@
             </xacro:cylinder_inertia>
         </link>
-        <joint name="${name}_rotation_joint" type="continuous">
+        <joint name="${name}_rotation_joint" type="fixed">
             <parent link="${robot_name}/base_link" />
             <child link="${name}_rotation_link" />
@@ -53,5 +53,5 @@
             <!-- <dynamics damping="0.00001" friction="1.0" /> -->
         </joint>
-        <joint name="${name}_wheel_joint" type="continuous">
+        <joint name="${name}_wheel_joint" type="fixed">
             <parent link="${name}_rotation_link" />
             <child link="${name}_wheel_link" />

File: vc200_description/urdf/parameters.xacro (robot description, xacro)
@@ -7,11 +7,11 @@
     <xacro:property name="chassis_length" value="0.355" />
     <xacro:property name="chassis_width" value="0.18" />
-    <xacro:property name="chassis_height" value="0.108" />
+    <xacro:property name="chassis_height" value="0.12" />
     <xacro:property name="chassis_mass" value="0.5" /> <!-- TODO -->
     <xacro:property name="clearence" value="0.042" />
     <xacro:property name="wheel_radius" value="0.0675" />
     <xacro:property name="wheel_mass" value="0.1" /> <!-- TODO -->
-    <xacro:property name="wheel_width" value="0.057" />
-    <xacro:property name="wheel_separation" value="0.3" />
+    <xacro:property name="wheel_width" value="0.06" />
+    <xacro:property name="wheel_separation" value="0.302" />
     <xacro:property name="wheelbase" value="0.24" />
     <xacro:property name="update_rate" value="50" />

File: vc200_description/urdf/vc200_description.xacro (robot description, xacro)
@@ -52,6 +52,4 @@
     <origin xyz="0.1 0.0 ${0.015+chassis_height+clearence}" rpy="0.0 0.0 0.0"/>
   </xacro:lidar>
-    <!-- radius="0.035"
-    length="0.0022"  -->
     <xacro:pozyx
       name="${robot_name}/pozyx"
@@ -66,16 +64,4 @@
       ay="0.0"
     />
-    <!-- <xacro:marvelmind
-      name="${robot_name}/marvelmind"
-      length ="0.055"
-      width ="0.055"
-      height ="0.033"
-      dx="0.1575"
-      dy="${-(chassis_width/2)+0.055/2+0.004}"
-      dz="0.14"
-      ar="0.0"
-      ap="0.69813170079"
-      ay="0.0"
-    /> -->
     <xacro:imu
       name="${robot_name}/stm_imu"
@@ -92,5 +78,4 @@
     <xacro:arg name="use_nominal_extrinsics" default="true" />
     <xacro:include filename="$(find vc200_description)/realsense2_description/urdf/_d435i.urdf.xacro"/>
-    <!-- <link name="base_link" /> -->
     <xacro:sensor_d435i parent="${robot_name}/base_footprint" use_nominal_extrinsics="$(arg use_nominal_extrinsics)">
       <origin xyz="${chassis_length/2 + 0.0149} 0 0.135" rpy="0 0 0"/>
