Commit message: Adding lidar, marvelmind, pozyx and camera description

File: vc200_description/urdf/macros/chassis.xacro (robot description, xacro)
@@ -1,10 +1,10 @@
 <?xml version="1.0"?>
 <robot xmlns:xacro="http://www.ros.org/wiki/xacro">
-    <xacro:macro name="chassis" params="name lenght width height clearence">
+    <xacro:macro name="chassis" params="name length width height clearence">
         <link name="${name}_link">
             <visual>
                 <origin xyz="0.0 0.0 ${height/2.0 + clearence}" rpy="0.0 0.0 0.0" />
                 <geometry>
-                    <box size="${lenght} ${width} ${height}" />
+                    <box size="${length} ${width} ${height}" />
                 </geometry>
                 <material name="chassis" />

File: vc200_description/urdf/macros/macros.xacro (robot description, xacro)
@@ -4,3 +4,6 @@
     <xacro:include filename="$(find vc200_description)/urdf/macros/wheel.xacro" />
     <xacro:include filename="$(find vc200_description)/urdf/macros/materials.xacro" />
+    <xacro:include filename="$(find vc200_description)/urdf/macros/pozyx.xacro" />
+    <xacro:include filename="$(find vc200_description)/urdf/macros/marvelmind.xacro" />
+    <xacro:include filename="$(find vc200_description)/urdf/macros/lidar.xacro" />
 </robot>

File: vc200_description/urdf/macros/materials.xacro (robot description, xacro)
@@ -7,3 +7,12 @@
         <color rgba="0 1 1 1.0"/>
     </material>
+    <material name="pozyx">
+        <color rgba="1 1 1 1.0"/>
+    </material>
+    <material name="marvelmind">
+        <color rgba="0 0 0 1.0"/>
+    </material>
+    <material name="lidar">
+        <color rgba="1 1 1 1.0"/>
+    </material>
 </robot>

File: vc200_description/urdf/parameters.xacro (robot description, xacro)
@@ -5,10 +5,12 @@
     <!-- Constants -->
     <xacro:property name="PI" value="3.1415926535897931" />
-    <xacro:property name="chassis_lenght" value="0.355" />
+    <xacro:property name="chassis_length" value="0.355" />
     <xacro:property name="chassis_width" value="0.18" />
     <xacro:property name="chassis_height" value="0.108" />
-    <xacro:property name="clearence" value="0.046" />
+    <xacro:property name="clearence" value="0.042" />
     <xacro:property name="wheel_radius" value="0.0675" />
     <xacro:property name="wheel_width" value="0.057" />
     <xacro:property name="wheel_separation" value="0.3"/>
+    <xacro:property name="wheelbase" value="0.24"/>
+    wheelbase
 </robot>

File: vc200_description/urdf/vc200_description.xacro (robot description, xacro)
@@ -1,4 +1,5 @@
 <?xml version="1.0"?>
-<robot name="$(arg robot_name)" xmlns:xacro="http://www.ros.org/wiki/xacro">
+<!-- <robot name="$(arg robot_name)" xmlns:xacro="http://www.ros.org/wiki/xacro"> -->
+<robot name="vc200" xmlns:xacro="http://www.ros.org/wiki/xacro">
     <xacro:include filename="$(find vc200_description)/urdf/parameters.xacro" />
     <xacro:include filename="$(find vc200_description)/urdf/macros/macros.xacro" />
@@ -6,5 +7,5 @@
     <xacro:chassis
       name="${robot_name}/base"
-      lenght="${chassis_lenght}"
+      length="${chassis_length}"
       width="${chassis_width}"
       height="${chassis_height}"
@@ -15,5 +16,5 @@
       radius="${wheel_radius}"
       width="${wheel_width}"
-      dx="${0.235/2.0}"
+      dx="${wheelbase/2.0}"
       dy="${wheel_separation/2.0}"
     />
@@ -22,5 +23,5 @@
       radius="${wheel_radius}"
       width="${wheel_width}"
-      dx="${0.235/2.0}"
+      dx="${wheelbase/2.0}"
       dy="-${wheel_separation/2.0}"
     />
@@ -29,5 +30,5 @@
       radius="${wheel_radius}"
       width="${wheel_width}"
-      dx="-${0.235/2.0}"
+      dx="-${wheelbase/2.0}"
       dy="${wheel_separation/2.0}"
     />
@@ -36,6 +37,46 @@
       radius="${wheel_radius}"
       width="${wheel_width}"
-      dx="-${0.235/2.0}"
+      dx="-${wheelbase/2.0}"
       dy="-${wheel_separation/2.0}"
     />
+    <xacro:lidar
+      name="${robot_name}/lidar"
+      radius="0.035"
+      length="0.022"
+      dx="0.0425"
+      dy="0.0"
+      dz="0.205"
+      ar="0.0"
+      ap="0.0"
+      ay="0.0"
+    />
+    <!-- radius="0.035"
+    length="0.0022"  -->
+    <xacro:pozyx
+      name="${robot_name}/pozyx"
+      length="0.008"
+      width="0.006"
+      height="0.003"
+      dx="-0.025"
+      dy="0.045"
+      dz="${0.12+clearence+0.003/3}"
+    />
+    <xacro:marvelmind
+      name="${robot_name}/marvelmind"
+      length ="0.055"
+      width ="0.055"
+      height ="0.033"
+      dx="0.1575"
+      dy="${-(chassis_width/2)+0.055/2+0.004}"
+      dz="0.14"
+      ar="0.0"
+      ap="0.69813170079"
+      ay="0.0"
+    />
+    <xacro:arg name="use_nominal_extrinsics" default="true" />
+    <xacro:include filename="$(find vc200_description)/realsense2_description/urdf/_d435i.urdf.xacro"/>
+    <!-- <link name="base_link" /> -->
+    <xacro:sensor_d435i parent="${robot_name}/base_footprint" use_nominal_extrinsics="$(arg use_nominal_extrinsics)">
+      <origin xyz="${chassis_length/2 + 0.0149} 0 0.135" rpy="0 0 0"/>
+    </xacro:sensor_d435i>
 </robot>

Commit message: extends the description of the robot and adds a simulation launcher

File: vc200_description/urdf/macros/chassis.xacro (robot description, xacro)
@@ -1,6 +1,12 @@
 <?xml version="1.0"?>
 <robot xmlns:xacro="http://www.ros.org/wiki/xacro">
-    <xacro:macro name="chassis" params="name length width height clearence">
+    <xacro:macro name="chassis" params="name length width height clearence mass">
         <link name="${name}_link">
+            <collision>
+                <origin xyz="0.0 0.0 ${height/2.0 + clearence}" rpy="0 0 0" />
+                <geometry>
+                    <box size="${length} ${width} ${height}" />
+                </geometry>
+            </collision>
             <visual>
                 <origin xyz="0.0 0.0 ${height/2.0 + clearence}" rpy="0.0 0.0 0.0" />
@@ -10,4 +16,7 @@
                 <material name="chassis" />
             </visual>
+            <xacro:cuboid_inertia x="${length}" y="${width}" z="${height}" mass="${mass}">
+                <origin xyz="0.0 0.0 ${height/2.0 + clearence}" rpy="0.0 0.0 0.0" />
+            </xacro:cuboid_inertia>
         </link>
         <joint name="${name}_joint" type="fixed">
@@ -15,4 +24,5 @@
             <child link="${name}_link" />
             <origin xyz="0 0 0" rpy="0 0 0" />
+            <axis xyz="0 1 0" rpy="0 0 0" />
         </joint>
     </xacro:macro>

File: vc200_description/urdf/macros/macros.xacro (robot description, xacro)
@@ -8,3 +8,5 @@
     <xacro:include filename="$(find vc200_description)/urdf/macros/lidar.xacro" />
     <xacro:include filename="$(find vc200_description)/urdf/macros/imu.xacro" />
+    <xacro:include filename="$(find vc200_description)/urdf/macros/caster_wheel.xacro" />
+    <xacro:include filename="$(find vc200_description)/urdf/macros/inertia.xacro" />
 </robot>

File: vc200_description/urdf/macros/materials.xacro (robot description, xacro)
@@ -19,3 +19,6 @@
         <color rgba="1 1 1 1.0"/>
     </material>
+    <material name="white">
+        <color rgba="1 1 1 1.0"/>
+    </material>
 </robot>

File: vc200_description/urdf/macros/wheel.xacro (robot description, xacro)
@@ -1,8 +1,8 @@
 <?xml version="1.0"?>
 <robot xmlns:xacro="http://www.ros.org/wiki/xacro">
-    <xacro:macro name="wheel" params="name radius width dx dy">
+    <xacro:macro name="wheel" params="name radius width dx dy mass">
         <link name="${name}_link">
-            <collision>
-                <origin xyz="0 0 0" rpy="0 0 0" />
+            <collision name="${name}">
+                <origin xyz="0 0 0" rpy="${PI/2} 0.0 0.0" />
                 <geometry>
                     <cylinder radius="${radius}" length="${width}" />
@@ -10,5 +10,5 @@
             </collision>
             <visual>
-                <origin xyz="0.0 0.0 0.0" rpy="0.0 0.0 0.0" />
+                <origin xyz="0.0 0.0 0.0" rpy="${PI/2} 0.0 0.0" />
                 <geometry>
                     <cylinder radius="${radius}" length="${width}" />
@@ -16,11 +16,24 @@
                 <material name="wheel" />
             </visual>
+            <xacro:cylinder_inertia radius="${radius}" length="${width}" mass="${mass}">
+                <origin xyz="0.0 0.0 0.0" rpy="${PI/2} 0.0 0.0"/>
+            </xacro:cylinder_inertia>
         </link>
         <joint name="${name}_joint" type="continuous">
-            <parent link="${robot_name}/base_footprint" />
+            <parent link="${robot_name}/base_link" />
             <child link="${name}_link" />
-            <origin xyz="${dx} ${dy} ${radius}" rpy="${-PI/2.0} 0 0" />
-            <axis xyz="0 0 1" />
+            <origin xyz="${dx} ${dy} ${radius}" rpy="0 0 0" />
+            <axis xyz="0 1 0" />
+            <dynamics damping="0.01" friction="5" />
         </joint>
+        <transmission name="${name}_trans">
+            <type>transmission_interface/SimpleTransmission</type>
+            <actuator name="${name}_motor">
+                <mechanicalReduction>1</mechanicalReduction>
+            </actuator>
+            <joint name="${name}_joint">
+                <hardwareInterface>hardware_interface/VelocityJointInterface</hardwareInterface>
+            </joint>
+        </transmission>
     </xacro:macro>
 </robot>

File: vc200_description/urdf/parameters.xacro (robot description, xacro)
@@ -8,8 +8,13 @@
     <xacro:property name="chassis_width" value="0.18" />
     <xacro:property name="chassis_height" value="0.108" />
+    <xacro:property name="chassis_mass" value="0.5" /> <!-- TODO -->
     <xacro:property name="clearence" value="0.042" />
     <xacro:property name="wheel_radius" value="0.0675" />
+    <xacro:property name="wheel_mass" value="0.1" /> <!-- TODO -->
     <xacro:property name="wheel_width" value="0.057" />
-    <xacro:property name="wheel_separation" value="0.3"/>
-    <xacro:property name="wheelbase" value="0.24"/>
+    <xacro:property name="wheel_separation" value="0.3" />
+    <xacro:property name="wheelbase" value="0.24" />
+    <xacro:property name="update_rate" value="50" />
+    <!-- <xacro:property name="odometry_source" value="encoder" /> -->
+    <xacro:property name="odometry_source" value="world" />
 </robot>

File: vc200_description/urdf/vc200_description.xacro (robot description, xacro)
@@ -1,5 +1,5 @@
 <?xml version="1.0"?>
-<robot name="$(arg robot_name)" xmlns:xacro="http://www.ros.org/wiki/xacro">
-<!-- <robot name="vc200" xmlns:xacro="http://www.ros.org/wiki/xacro"> -->
+<!-- <robot name="$(arg robot_name)" xmlns:xacro="http://www.ros.org/wiki/xacro"> -->
+<robot name="vc200" xmlns:xacro="http://www.ros.org/wiki/xacro">
     <xacro:include filename="$(find vc200_description)/urdf/parameters.xacro" />
     <xacro:include filename="$(find vc200_description)/urdf/macros/macros.xacro" />
@@ -11,4 +11,5 @@
       height="${chassis_height}"
       clearence="${clearence}"
+      mass="${chassis_mass}"
     />
     <xacro:wheel
@@ -16,4 +17,5 @@
       radius="${wheel_radius}"
       width="${wheel_width}"
+      mass="${wheel_mass}"
       dx="${wheelbase/2.0}"
       dy="${wheel_separation/2.0}"
@@ -23,20 +25,25 @@
       radius="${wheel_radius}"
       width="${wheel_width}"
+      mass="${wheel_mass}"
       dx="${wheelbase/2.0}"
       dy="-${wheel_separation/2.0}"
     />
-    <xacro:wheel
-      name="${robot_name}/rear_left_wheel"
-      radius="${wheel_radius}"
-      width="${wheel_width}"
-      dx="-${wheelbase/2.0}"
-      dy="${wheel_separation/2.0}"
+    <xacro:caster_wheel
+      name="${robot_name}/swivel_wheel_right"
+      radius="0.0125"
+      mass="0.01"
+      dx="-0.15"
+      dy="-0.05"
+      offset="0.014"
+      width="0.028"
     />
-    <xacro:wheel
-      name="${robot_name}/rear_right_wheel"
-      radius="${wheel_radius}"
-      width="${wheel_width}"
-      dx="-${wheelbase/2.0}"
-      dy="-${wheel_separation/2.0}"
+    <xacro:caster_wheel
+      name="${robot_name}/swivel_wheel_left"
+      radius="0.0125"
+      mass="0.01"
+      dx="-0.15"
+      dy="0.05"
+      offset="0.014"
+      width="0.028"
     />
     <xacro:lidar
@@ -65,5 +72,5 @@
       ay="0.0"
     />
-    <xacro:marvelmind
+    <!-- <xacro:marvelmind
       name="${robot_name}/marvelmind"
       length ="0.055"
@@ -76,5 +83,5 @@
       ap="0.69813170079"
       ay="0.0"
-    />
+    /> -->
     <xacro:imu
       name="${robot_name}/stm_imu"

Commit message: Change of base_footprint location

File: vc200_description/urdf/macros/chassis.xacro (robot description, xacro)
@@ -1,8 +1,8 @@
 <?xml version="1.0"?>
 <robot xmlns:xacro="http://www.ros.org/wiki/xacro">
-    <xacro:macro name="chassis" params="name length width height clearence mass">
+    <xacro:macro name="chassis" params="name length width height clearence offset mass">
         <link name="${name}_link">
             <collision>
-                <origin xyz="0.0 0.0 ${height/2.0 + clearence}" rpy="0 0 0" />
+                <origin xyz="${offset} 0.0 ${height/2.0 + clearence}" rpy="0 0 0" />
                 <geometry>
                     <box size="${length} ${width} ${height}" />
@@ -10,5 +10,5 @@
             </collision>
             <visual>
-                <origin xyz="0.0 0.0 ${height/2.0 + clearence}" rpy="0.0 0.0 0.0" />
+                <origin xyz="${offset} 0.0 ${height/2.0 + clearence}" rpy="0.0 0.0 0.0" />
                 <geometry>
                     <box size="${length} ${width} ${height}" />
@@ -17,5 +17,5 @@
             </visual>
             <xacro:cuboid_inertia x="${length}" y="${width}" z="${height}" mass="${mass}">
-                <origin xyz="0.0 0.0 ${height/2.0 + clearence}" rpy="0.0 0.0 0.0" />
+                <origin xyz="${offset} 0.0 ${height/2.0 + clearence}" rpy="0.0 0.0 0.0" />
             </xacro:cuboid_inertia>
         </link>
@@ -23,5 +23,5 @@
             <parent link="${robot_name}/base_footprint" />
             <child link="${name}_link" />
-            <origin xyz="0 0 0" rpy="0 0 0" />
+            <origin xyz="${offset} 0 0" rpy="0 0 0" />
             <axis xyz="0 1 0" rpy="0 0 0" />
         </joint>

File: vc200_description/urdf/vc200_description.xacro (robot description, xacro)
@@ -1,5 +1,5 @@
 <?xml version="1.0"?>
-<robot name="$(arg robot_name)" xmlns:xacro="http://www.ros.org/wiki/xacro">
-<!-- <robot name="vc200" xmlns:xacro="http://www.ros.org/wiki/xacro"> -->
+<!-- <robot name="$(arg robot_name)" xmlns:xacro="http://www.ros.org/wiki/xacro"> -->
+<robot name="vc200" xmlns:xacro="http://www.ros.org/wiki/xacro">
     <xacro:include filename="$(find vc200_description)/urdf/parameters.xacro" />
     <xacro:include filename="$(find vc200_description)/urdf/macros/macros.xacro" />
@@ -11,4 +11,5 @@
       height="${chassis_height}"
       clearence="${clearence}"
+      offset="${-wheelbase/4.0}"
       mass="${chassis_mass}"
     />
@@ -18,5 +19,5 @@
       width="${wheel_width}"
       mass="${wheel_mass}"
-      dx="${wheelbase/2.0}"
+      dx="${wheelbase/4.0}"
       dy="${wheel_separation/2.0}"
     />
@@ -26,5 +27,5 @@
       mass="${wheel_mass}"
       width="${wheel_width}"
-      dx="${wheelbase/2.0}"
+      dx="${wheelbase/4.0}"
       dy="-${wheel_separation/2.0}"
     />
@@ -32,5 +33,5 @@
     radius="0.0125"
     mass="0.01"
-    dx="-0.15"
+    dx="${-wheelbase/4.0 -0.15}"
     dy="-0.05"
     offset="0.014"
@@ -40,5 +41,5 @@
     radius="0.0125"
     mass="0.01"
-    dx="-0.15"
+    dx="${-wheelbase/4.0 -0.15}"
     dy="0.05"
     offset="0.014"
@@ -50,5 +51,5 @@
     height="0.03"
     mass="0.17" >
-    <origin xyz="0.1 0.0 ${0.015+chassis_height+clearence}" rpy="0.0 0.0 0.0"/>
+    <origin xyz="${-0.009} 0.0 ${0.015+chassis_height+clearence}" rpy="0.0 0.0 0.0"/>
   </xacro:lidar>
     <xacro:pozyx
@@ -57,5 +58,5 @@
       width="0.006"
       height="0.003"
-      dx="-0.025"
+      dx="${-0.025-wheelbase/2.0}"
       dy="0.045"
       dz="${0.12+clearence+0.003/2}"
@@ -69,5 +70,5 @@
       width="0.006"
       height="0.003"
-      dx="-0.025"
+      dx="${-0.025 -wheelbase/2.0}"
       dy="0.045"
       dz="${0.12+clearence+0.003/2 - 0.02}"
@@ -79,5 +80,5 @@
     <xacro:include filename="$(find vc200_description)/realsense2_description/urdf/_d435i.urdf.xacro"/>
     <xacro:sensor_d435i parent="${robot_name}/base_footprint" use_nominal_extrinsics="$(arg use_nominal_extrinsics)">
-      <origin xyz="${chassis_length/2 + 0.0149} 0 0.135" rpy="0 0 0"/>
+      <origin xyz="${chassis_length/2 + 0.0149 -wheelbase/2.0} 0 0.135" rpy="0 0 0"/>
     </xacro:sensor_d435i>
 </robot>
