Commit message: diff drive parameters setup

File: vc200_description/urdf/parameters.xacro (robot description, xacro)
@@ -9,6 +9,6 @@
     <xacro:property name="chassis_height" value="0.108" />
     <xacro:property name="clearence" value="0.046" />
-    <xacro:property name="wheel_radius" value="0.065" />
-    <xacro:property name="wheel_width" value="0.04" />
-    <xacro:property name="wheel_separation" value="0.25"/>
+    <xacro:property name="wheel_radius" value="0.0675" />
+    <xacro:property name="wheel_width" value="0.057" />
+    <xacro:property name="wheel_separation" value="0.3"/>
 </robot>

File: vc200_description/urdf/vc200_description.xacro (robot description, xacro)
@@ -15,5 +15,5 @@
       radius="${wheel_radius}"
       width="${wheel_width}"
-      dx="0.1125"
+      dx="${0.235/2.0}"
       dy="${wheel_separation/2.0}"
     />
@@ -22,5 +22,5 @@
       radius="${wheel_radius}"
       width="${wheel_width}"
-      dx="0.1125"
+      dx="${0.235/2.0}"
       dy="-${wheel_separation/2.0}"
     />
@@ -29,5 +29,5 @@
       radius="${wheel_radius}"
       width="${wheel_width}"
-      dx="-0.1125"
+      dx="-${0.235/2.0}"
       dy="${wheel_separation/2.0}"
     />
@@ -36,5 +36,5 @@
       radius="${wheel_radius}"
       width="${wheel_width}"
-      dx="-0.1125"
+      dx="-${0.235/2.0}"
       dy="-${wheel_separation/2.0}"
     />

Commit message: description update

File: vc200_description/urdf/parameters.xacro (robot description, xacro)
@@ -13,5 +13,5 @@
     <xacro:property name="wheel_mass" value="0.1" /> <!-- TODO -->
     <xacro:property name="wheel_width" value="0.06" />
-    <xacro:property name="wheel_separation" value="0.302" />
+    <xacro:property name="wheel_separation" value="0.31" />
     <xacro:property name="wheelbase" value="0.24" />
     <xacro:property name="update_rate" value="50" />

File: vc200_description/urdf/vc200_description.xacro (robot description, xacro)
@@ -51,5 +51,5 @@
     height="0.03"
     mass="0.17" >
-    <origin xyz="${-0.009} 0.0 ${0.015+chassis_height+clearence}" rpy="0.0 0.0 0.0"/>
+    <origin xyz="${-0.009} 0.0 ${0.015+chassis_height+clearence}" rpy="0.0 0.0 ${PI}"/>
   </xacro:lidar>
     <xacro:pozyx
